File: SmartReel.kicad_pcb (KiCad board)
At the start: 2 copper layers, 64.3 x 74 mm, 42 parts, among them J1 8 pin header, J2 8 pin socket, SW1 Switch, SW2 Switch, SW3 Switch, SW4 Switch, U1 74HC14, U2 Photointerrupter, U3 Photointerrupter, U4 Photointerrupter, U5 Photointerrupter, U6 74HC165

Commit message: Commit to upload
Parts:
- removed C1, C10, C2, C3, C4, C5, C6, C7, C8, C9: 100n, Capacitor_SMD:C_0402_1005Metric
- removed D1, D2, D3, D4: WS2812B, LED_SMD:LED_WS2812B_PLCC4_5.0x5.0mm_P3.2mm
- removed H1, H2: MountingHole, MountingHole:MountingHole_5.3mm_M5_Pad_TopBottom
- removed R1, R11, R2, R3, R4, R6, R7, R9: 10k, Resistor_SMD:R_0402_1005Metric
- removed R10, R12, R5, R8: 330, Resistor_SMD:R_0402_1005Metric
- removed SW1, SW2, SW3, SW4: Switch, EasyEDA_Lib:SW-TH_SHOU-HAN_3JWD-DBHD-13.5
- removed U1: 74HC14, Package_SO:SOIC-14_3.9x8.7mm_P1.27mm
- removed U6: 74HC165, Package_SO:SOIC-16_3.9x9.9mm_P1.27mm
- added C11: 100n, Capacitor_SMD:C_0402_1005Metric, B.Cu at (91.3, 115.2)
- added C12: 100n, Capacitor_SMD:C_0402_1005Metric, B.Cu at (31.3, 115.2)
- added C19: 100n, Capacitor_SMD:C_0402_1005Metric, B.Cu at (105.8, 115.2)
- added C20: 100n, Capacitor_SMD:C_0402_1005Metric, B.Cu at (120.8, 115.2)
- added C21: 100n, Capacitor_SMD:C_0402_1005Metric, B.Cu at (135.8, 115.3)
- added C22: 100n, Capacitor_SMD:C_0402_1005Metric, F.Cu at (118.5, 66.1)
- added C23: 100n, Capacitor_SMD:C_0402_1005Metric, B.Cu at (135.1, 77.8)
- added C24: 100n, Capacitor_SMD:C_0402_1005Metric, B.Cu at (138.5, 97.9)
- added C25: 100n, Capacitor_SMD:C_0402_1005Metric, B.Cu at (90.1, 77.8)
- added C26: 100n, Capacitor_SMD:C_0402_1005Metric, B.Cu at (93.5, 97.9)
- added C27: 100n, Capacitor_SMD:C_0402_1005Metric, B.Cu at (105.1, 77.8)
- added C28: 100n, Capacitor_SMD:C_0402_1005Metric, B.Cu at (108.5, 97.9)
- added C29: 100n, Capacitor_SMD:C_0402_1005Metric, B.Cu at (120.1, 77.8)
- added C30: 100n, Capacitor_SMD:C_0402_1005Metric, B.Cu at (123.5, 97.9)
- added C31: 100n, Capacitor_SMD:C_0402_1005Metric, B.Cu at (151.3, 115.2)
- added C32: 100n, Capacitor_SMD:C_0402_1005Metric, B.Cu at (165.8, 115.2)
- added C33: 100n, Capacitor_SMD:C_0402_1005Metric, B.Cu at (180.8, 115.2)
- added C34: 100n, Capacitor_SMD:C_0402_1005Metric, B.Cu at (195.8, 115.3)
- added C35: 100n, Capacitor_SMD:C_0402_1005Metric, F.Cu at (178.5, 66.1)
- added C36: 100n, Capacitor_SMD:C_0402_1005Metric, B.Cu at (195.1, 77.8)
- added C37: 100n, Capacitor_SMD:C_0402_1005Metric, B.Cu at (198.5, 97.9)
- added C38: 100n, Capacitor_SMD:C_0402_1005Metric, B.Cu at (150.1, 77.8)
- added C39: 100n, Capacitor_SMD:C_0402_1005Metric, B.Cu at (153.5, 97.9)
- added C40: 100n, Capacitor_SMD:C_0402_1005Metric, B.Cu at (165.1, 77.8)
- added C41: 100n, Capacitor_SMD:C_0402_1005Metric, B.Cu at (168.5, 97.9)
- added C42: 100n, Capacitor_SMD:C_0402_1005Metric, B.Cu at (180.1, 77.8)
- added C43: 100n, Capacitor_SMD:C_0402_1005Metric, B.Cu at (183.5, 97.9)
- added C44: 100n, Capacitor_SMD:C_0402_1005Metric, B.Cu at (211.3, 115.2)
- added C45: 100n, Capacitor_SMD:C_0402_1005Metric, B.Cu at (225.8, 115.2)
- added C46: 100n, Capacitor_SMD:C_0402_1005Metric, B.Cu at (240.8, 115.2)
- added C47: 100n, Capacitor_SMD:C_0402_1005Metric, B.Cu at (255.8, 115.3)
- added C48: 100n, Capacitor_SMD:C_0402_1005Metric, F.Cu at (238.5, 66.1)
- added C49: 100n, Capacitor_SMD:C_0402_1005Metric, B.Cu at (255.1, 77.8)
- added C50: 100n, Capacitor_SMD:C_0402_1005Metric, B.Cu at (258.5, 97.9)
- added C51: 100n, Capacitor_SMD:C_0402_1005Metric, B.Cu at (210.1, 77.8)
- added C52: 100n, Capacitor_SMD:C_0402_1005Metric, B.Cu at (213.5, 97.9)
- added C53: 100n, Capacitor_SMD:C_0402_1005Metric, B.Cu at (225.1, 77.8)
- added C54: 100n, Capacitor_SMD:C_0402_1005Metric, B.Cu at (228.5, 97.9)
- added C55: 100n, Capacitor_SMD:C_0402_1005Metric, B.Cu at (240.1, 77.8)
- added C56: 100n, Capacitor_SMD:C_0402_1005Metric, B.Cu at (243.5, 97.9)
- added C57: 100n, Capacitor_SMD:C_0402_1005Metric, B.Cu at (45.8, 115.2)
- added C58: 100n, Capacitor_SMD:C_0402_1005Metric, B.Cu at (60.8, 115.2)
- added C59: 100n, Capacitor_SMD:C_0402_1005Metric, B.Cu at (75.8, 115.3)
- added C60: 100n, Capacitor_SMD:C_0402_1005Metric, F.Cu at (58.5, 66.1)
- added C61: 100n, Capacitor_SMD:C_0402_1005Metric, B.Cu at (75.1, 77.8)
- added C62: 100n, Capacitor_SMD:C_0402_1005Metric, B.Cu at (78.5, 97.9)
- added C63: 100n, Capacitor_SMD:C_0402_1005Metric, B.Cu at (30.1, 77.8)
- added C64: 100n, Capacitor_SMD:C_0402_1005Metric, B.Cu at (33.5, 97.9)
- added C65: 100n, Capacitor_SMD:C_0402_1005Metric, B.Cu at (45.1, 77.8)
- added C66: 100n, Capacitor_SMD:C_0402_1005Metric, B.Cu at (48.5, 97.9)
- added C67: 100n, Capacitor_SMD:C_0402_1005Metric, B.Cu at (60.1, 77.8)
- added C68: 100n, Capacitor_SMD:C_0402_1005Metric, B.Cu at (63.5, 97.9)
- added CN1: M3 Solder Nut, EasyEDA_Lib:M3-TH_BD6.0-D4.3, F.Cu at (33.2, 49.2)
- added CN2: M3 Solder Nut, EasyEDA_Lib:M3-TH_BD6.0-D4.3, F.Cu at (147.0, 49.2)
- added CN3: M3 Solder Nut, EasyEDA_Lib:M3-TH_BD6.0-D4.3, F.Cu at (260.7, 49.2)
- added D10: WS2812B, LED_SMD:LED_WS2812B_PLCC4_5.0x5.0mm_P3.2mm, B.Cu at (165.7, 119.5)
- added D11: WS2812B, LED_SMD:LED_WS2812B_PLCC4_5.0x5.0mm_P3.2mm, B.Cu at (180.7, 119.5)
- added D12: WS2812B, LED_SMD:LED_WS2812B_PLCC4_5.0x5.0mm_P3.2mm, B.Cu at (195.7, 119.5)
- added D13: WS2812B, LED_SMD:LED_WS2812B_PLCC4_5.0x5.0mm_P3.2mm, B.Cu at (211.2, 119.5)
- added D14: WS2812B, LED_SMD:LED_WS2812B_PLCC4_5.0x5.0mm_P3.2mm, B.Cu at (225.7, 119.5)
- added D15: WS2812B, LED_SMD:LED_WS2812B_PLCC4_5.0x5.0mm_P3.2mm, B.Cu at (240.7, 119.5)
- added D16: WS2812B, LED_SMD:LED_WS2812B_PLCC4_5.0x5.0mm_P3.2mm, B.Cu at (255.7, 119.5)
- added D17: WS2812B, LED_SMD:LED_WS2812B_PLCC4_5.0x5.0mm_P3.2mm, B.Cu at (31.2, 119.5)
- added D18: WS2812B, LED_SMD:LED_WS2812B_PLCC4_5.0x5.0mm_P3.2mm, B.Cu at (45.7, 119.5)
- added D19: WS2812B, LED_SMD:LED_WS2812B_PLCC4_5.0x5.0mm_P3.2mm, B.Cu at (60.7, 119.5)
- added D20: WS2812B, LED_SMD:LED_WS2812B_PLCC4_5.0x5.0mm_P3.2mm, B.Cu at (75.7, 119.5)
- added D5: WS2812B, LED_SMD:LED_WS2812B_PLCC4_5.0x5.0mm_P3.2mm, B.Cu at (91.2, 119.5)
- added D6: WS2812B, LED_SMD:LED_WS2812B_PLCC4_5.0x5.0mm_P3.2mm, B.Cu at (105.7, 119.5)
- added D7: WS2812B, LED_SMD:LED_WS2812B_PLCC4_5.0x5.0mm_P3.2mm, B.Cu at (120.7, 119.5)
- added D8: WS2812B, LED_SMD:LED_WS2812B_PLCC4_5.0x5.0mm_P3.2mm, B.Cu at (135.7, 119.5)
- added D9: WS2812B, LED_SMD:LED_WS2812B_PLCC4_5.0x5.0mm_P3.2mm, B.Cu at (151.2, 119.5)
- added H11: MountingHole, MountingHole:MountingHole_5.3mm_M5, F.Cu at (143.2, 114.2)
- added H12: MountingHole, MountingHole:MountingHole_5.3mm_M5, F.Cu at (248.2, 114.2)
- added H9: M5 Mounting Hole, MountingHole:MountingHole_5.3mm_M5, F.Cu at (38.2, 114.2)
- added R13: 10k, Resistor_SMD:R_0402_1005Metric, B.Cu at (136.4, 77.8)
- added R14: 10k, Resistor_SMD:R_0402_1005Metric, B.Cu at (138.5, 96.4)
- added R15: 10k, Resistor_SMD:R_0402_1005Metric, B.Cu at (91.4, 77.8)
- added R16: 10k, Resistor_SMD:R_0402_1005Metric, B.Cu at (93.5, 96.4)
- added R17: 10k, Resistor_SMD:R_0402_1005Metric, B.Cu at (106.4, 77.8)
- added R18: 10k, Resistor_SMD:R_0402_1005Metric, B.Cu at (108.5, 96.4)
- added R19: 10k, Resistor_SMD:R_0402_1005Metric, B.Cu at (121.4, 77.8)
- added R20: 10k, Resistor_SMD:R_0402_1005Metric, B.Cu at (123.5, 96.4)
- added R21: 10k, Resistor_SMD:R_0402_1005Metric, B.Cu at (196.4, 77.8)
- added R22: 10k, Resistor_SMD:R_0402_1005Metric, B.Cu at (198.5, 96.4)
- added R23: 10k, Resistor_SMD:R_0402_1005Metric, B.Cu at (151.4, 77.8)
- added R24: 10k, Resistor_SMD:R_0402_1005Metric, B.Cu at (153.5, 96.4)
- added R25: 10k, Resistor_SMD:R_0402_1005Metric, B.Cu at (166.4, 77.8)
- added R26: 10k, Resistor_SMD:R_0402_1005Metric, B.Cu at (168.5, 96.4)
- added R27: 10k, Resistor_SMD:R_0402_1005Metric, B.Cu at (181.4, 77.8)
- added R28: 10k, Resistor_SMD:R_0402_1005Metric, B.Cu at (183.5, 96.4)
- added R29: 10k, Resistor_SMD:R_0402_1005Metric, B.Cu at (256.4, 77.8)
- added R30: 10k, Resistor_SMD:R_0402_1005Metric, B.Cu at (258.5, 96.4)
- added R31: 10k, Resistor_SMD:R_0402_1005Metric, B.Cu at (211.4, 77.8)
- added R32: 10k, Resistor_SMD:R_0402_1005Metric, B.Cu at (213.5, 96.4)
- added R33: 10k, Resistor_SMD:R_0402_1005Metric, B.Cu at (226.4, 77.8)
- added R34: 10k, Resistor_SMD:R_0402_1005Metric, B.Cu at (228.5, 96.4)
- added R35: 10k, Resistor_SMD:R_0402_1005Metric, B.Cu at (241.4, 77.8)
- added R36: 10k, Resistor_SMD:R_0402_1005Metric, B.Cu at (243.5, 96.4)
- added R37: 10k, Resistor_SMD:R_0402_1005Metric, B.Cu at (76.4, 77.8)
- added R38: 10k, Resistor_SMD:R_0402_1005Metric, B.Cu at (78.5, 96.4)
- added R39: 10k, Resistor_SMD:R_0402_1005Metric, B.Cu at (31.4, 77.8)
- added R40: 10k, Resistor_SMD:R_0402_1005Metric, B.Cu at (33.5, 96.4)
- added R41: 10k, Resistor_SMD:R_0402_1005Metric, B.Cu at (46.4, 77.8)
- added R42: 10k, Resistor_SMD:R_0402_1005Metric, B.Cu at (48.5, 96.4)
- added R43: 10k, Resistor_SMD:R_0402_1005Metric, B.Cu at (61.4, 77.8)
- added R44: 10k, Resistor_SMD:R_0402_1005Metric, B.Cu at (63.5, 96.4)
- added SW13: Switch, EasyEDA_Lib:SW-TH_SHOU-HAN_3JWD-DBHD-13.5, F.Cu at (135.7, 85.8)
- added SW14: Switch, EasyEDA_Lib:SW-TH_SHOU-HAN_3JWD-DBHD-13.5, F.Cu at (143.2, 92.8)
- added SW15: Switch, EasyEDA_Lib:SW-TH_SHOU-HAN_3JWD-DBHD-13.5, F.Cu at (90.7, 85.8)
- added SW16: Switch, EasyEDA_Lib:SW-TH_SHOU-HAN_3JWD-DBHD-13.5, F.Cu at (98.2, 92.8)
- added SW17: Switch, EasyEDA_Lib:SW-TH_SHOU-HAN_3JWD-DBHD-13.5, F.Cu at (105.7, 85.8)
- added SW18: Switch, EasyEDA_Lib:SW-TH_SHOU-HAN_3JWD-DBHD-13.5, F.Cu at (113.2, 92.8)
- added SW19: Switch, EasyEDA_Lib:SW-TH_SHOU-HAN_3JWD-DBHD-13.5, F.Cu at (120.7, 85.8)
- added SW20: Switch, EasyEDA_Lib:SW-TH_SHOU-HAN_3JWD-DBHD-13.5, F.Cu at (128.2, 92.8)
- added SW21: Switch, EasyEDA_Lib:SW-TH_SHOU-HAN_3JWD-DBHD-13.5, F.Cu at (195.7, 85.8)
- added SW22: Switch, EasyEDA_Lib:SW-TH_SHOU-HAN_3JWD-DBHD-13.5, F.Cu at (203.2, 92.8)
- added SW23: Switch, EasyEDA_Lib:SW-TH_SHOU-HAN_3JWD-DBHD-13.5, F.Cu at (150.7, 85.8)
- added SW24: Switch, EasyEDA_Lib:SW-TH_SHOU-HAN_3JWD-DBHD-13.5, F.Cu at (158.2, 92.8)
- added SW25: Switch, EasyEDA_Lib:SW-TH_SHOU-HAN_3JWD-DBHD-13.5, F.Cu at (165.7, 85.8)
- added SW26: Switch, EasyEDA_Lib:SW-TH_SHOU-HAN_3JWD-DBHD-13.5, F.Cu at (173.2, 92.8)
- added SW27: Switch, EasyEDA_Lib:SW-TH_SHOU-HAN_3JWD-DBHD-13.5, F.Cu at (180.7, 85.8)
- added SW28: Switch, EasyEDA_Lib:SW-TH_SHOU-HAN_3JWD-DBHD-13.5, F.Cu at (188.2, 92.8)
- added SW29: Switch, EasyEDA_Lib:SW-TH_SHOU-HAN_3JWD-DBHD-13.5, F.Cu at (255.7, 85.8)
- added SW30: Switch, EasyEDA_Lib:SW-TH_SHOU-HAN_3JWD-DBHD-13.5, F.Cu at (263.2, 92.8)
- added SW31: Switch, EasyEDA_Lib:SW-TH_SHOU-HAN_3JWD-DBHD-13.5, F.Cu at (210.7, 85.8)
- added SW32: Switch, EasyEDA_Lib:SW-TH_SHOU-HAN_3JWD-DBHD-13.5, F.Cu at (218.2, 92.8)
- added SW33: Switch, EasyEDA_Lib:SW-TH_SHOU-HAN_3JWD-DBHD-13.5, F.Cu at (225.7, 85.8)
- added SW34: Switch, EasyEDA_Lib:SW-TH_SHOU-HAN_3JWD-DBHD-13.5, F.Cu at (233.2, 92.8)
- added SW35: Switch, EasyEDA_Lib:SW-TH_SHOU-HAN_3JWD-DBHD-13.5, F.Cu at (240.7, 85.8)
- added SW36: Switch, EasyEDA_Lib:SW-TH_SHOU-HAN_3JWD-DBHD-13.5, F.Cu at (248.2, 92.8)
- added SW37: Switch, EasyEDA_Lib:SW-TH_SHOU-HAN_3JWD-DBHD-13.5, F.Cu at (75.7, 85.8)
- added SW38: Switch, EasyEDA_Lib:SW-TH_SHOU-HAN_3JWD-DBHD-13.5, F.Cu at (83.2, 92.8)
- added SW39: Switch, EasyEDA_Lib:SW-TH_SHOU-HAN_3JWD-DBHD-13.5, F.Cu at (30.7, 85.8)
- added SW40: Switch, EasyEDA_Lib:SW-TH_SHOU-HAN_3JWD-DBHD-13.5, F.Cu at (38.2, 92.8)
- added SW41: Switch, EasyEDA_Lib:SW-TH_SHOU-HAN_3JWD-DBHD-13.5, F.Cu at (45.7, 85.8)
- added SW42: Switch, EasyEDA_Lib:SW-TH_SHOU-HAN_3JWD-DBHD-13.5, F.Cu at (53.2, 92.8)
- added SW43: Switch, EasyEDA_Lib:SW-TH_SHOU-HAN_3JWD-DBHD-13.5, F.Cu at (60.7, 85.8)
- added SW44: Switch, EasyEDA_Lib:SW-TH_SHOU-HAN_3JWD-DBHD-13.5, F.Cu at (68.2, 92.8)
- U2, U3, U4, U5: value Photointerrupter -> 74HC165; footprint EasyEDA_Lib:OPTO-TH_ZGY8402-ITR -> Package_SO:SOIC-16_3.9x9.9mm_P1.27mm
- moved JP1 146.5 mm to (249.3, 55.5)
- moved U4 143.7 mm to (238.7, 58.1)
- moved J2 133.1 mm to (256.9, 66.0)
- moved U3 106.2 mm to (178.7, 58.1)
- moved U5 96.3 mm to (58.7, 58.1)
- moved U2 77.1 mm to (118.7, 58.1)
- moved J1 47.7 mm to (31.7, 66.0)
- moved P1 44.6 mm to (49.7, 55.2)
Connections:
- U2 pad 1: Net-(R5-Pad2) -> /SLATCH
- U2 pad 2: Earth -> /SCLK
- U2 pad 3: /OPT_CH1 -> /4 Switch Unit1/SW_CH3A
- U2 pad 4: Earth -> /4 Switch Unit1/SW_CH3B
- U3 pad 1: Net-(R8-Pad2) -> /SLATCH
- U3 pad 2: Earth -> /SCLK
- U3 pad 3: /OPT_CH2 -> /4 Switch Unit2/SW_CH3A
- U3 pad 4: Earth -> /4 Switch Unit2/SW_CH3B
- U4 pad 1: Net-(R10-Pad2) -> /SLATCH
- U4 pad 2: Earth -> /SCLK
- U4 pad 3: /OPT_CH3 -> /4 Switch Unit3/SW_CH3A
- U4 pad 4: Earth -> /4 Switch Unit3/SW_CH3B
- U5 pad 1: Net-(R12-Pad2) -> /SLATCH
- U5 pad 2: Earth -> /SCLK
- U5 pad 3: /OPT_CH4 -> /4 Switch Unit0/SW_CH3A
- U5 pad 4: Earth -> /4 Switch Unit0/SW_CH3B
Routing:
- net (no net): track 0.00 -> 46.3 mm, vias 0 -> 60
- net Earth: track 0.00 -> 25.2 mm, vias 0 -> 32
- net +5V: track 0.00 -> 24.2 mm, vias 0 -> 32
- net /4 Switch Unit3/SW_CH4B: track 0.00 -> 5.72 mm
- net /4 Switch Unit1/SW_CH3B: track 0.00 -> 5.72 mm
- net /4 Switch Unit1/SW_CH2B: track 0.00 -> 5.72 mm
- net /4 Switch Unit1/SW_CH1B: track 0.00 -> 5.72 mm
- net /4 Switch Unit0/SW_CH4B: track 0.00 -> 5.72 mm
- net /4 Switch Unit0/SW_CH3B: track 0.00 -> 5.72 mm
- net /4 Switch Unit3/SW_CH3B: track 0.00 -> 5.72 mm
- net /4 Switch Unit3/SW_CH2B: track 0.00 -> 5.72 mm
- net /4 Switch Unit3/SW_CH1B: track 0.00 -> 5.72 mm
- net /4 Switch Unit2/SW_CH3B: track 0.00 -> 5.72 mm
- net /4 Switch Unit2/SW_CH4B: track 0.00 -> 5.72 mm
- net /4 Switch Unit2/SW_CH2B: track 0.00 -> 5.72 mm
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Other:
- board size 64.3 x 74 mm -> 238.5 x 80 mm
- copper layers 2 -> 4
