File: SmartReel.kicad_sch (KiCad schematic)
At the start: 42 parts, among them J1 8 pin header, J2 8 pin socket, SW1 Switch, SW2 Switch, SW3 Switch, SW4 Switch, U1 74HC14, U2 Photointerrupter, U3 Photointerrupter, U4 Photointerrupter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

Commit message: Commit to upload
Parts:
- removed C1, C2, C3, C4: 100n, Capacitor_SMD:C_0402_1005Metric, symbol Device:C
- removed C10, C5, C6, C7, C8, C9: 100n, Capacitor_SMD:C_0402_1005Metric, symbol Device:C_Small
- removed D1, D2, D3, D4: WS2812B, LED_SMD:LED_WS2812B_PLCC4_5.0x5.0mm_P3.2mm, symbol LED:WS2812B
- removed H2: MountingHole, MountingHole:MountingHole_5.3mm_M5_Pad_TopBottom, symbol Mechanical:MountingHole
- removed R1, R11, R2, R3, R4, R6, R7, R9: 10k, Resistor_SMD:R_0402_1005Metric, symbol Device:R
- removed R10, R12, R5, R8: 330, Resistor_SMD:R_0402_1005Metric, symbol Device:R
- removed SW1, SW2, SW3, SW4: Switch, EasyEDA_Lib:SW-TH_SHOU-HAN_3JWD-DBHD-13.5, symbol EasyEDA_Lib:3JWD-DBHD-13.5 125
- removed U1: 74HC14, Package_SO:SOIC-14_3.9x8.7mm_P1.27mm, symbol EasyEDA_Lib:74HC14D,653
- removed U2, U3, U4, U5: Photointerrupter, EasyEDA_Lib:OPTO-TH_ZGY8402-ITR, symbol EasyEDA_Lib:ZGY8402(ITR)
- removed U6: 74HC165, Package_SO:SOIC-16_3.9x9.9mm_P1.27mm, symbol EasyEDA_Lib:74HC165D,653
- added CN1, CN2, CN3: M3 Solder Nut, EasyEDA_Lib:M3-TH_BD6.0-D4.3, symbol EasyEDA_Lib:SMTSOM330BTR
- added H11, H12: MountingHole, MountingHole:MountingHole_5.3mm_M5, symbol Mechanical:MountingHole
- H9: renamed from H1; value MountingHole -> M5 Mounting Hole; footprint MountingHole:MountingHole_5.3mm_M5_Pad_TopBottom -> MountingHole:MountingHole_5.3mm_M5
Connections:
- no-connect marks 7 -> 3
Other:
- added sheet 4 Switch Unit0 (Switch_Unit.kicad_sch)
- added sheet 4 Switch Unit1 (Switch_Unit.kicad_sch)
- added sheet 4 Switch Unit2 (Switch_Unit.kicad_sch)
- added sheet 4 Switch Unit3 (Switch_Unit.kicad_sch)
- moved on the sheet: H9, J1, J2
