File: ReelPCB/SmartReel.kicad_pcb (KiCad board)
At the start: 4 copper layers, 238.5 x 80 mm, 146 parts, among them CN1 M3 Solder Nut, CN2 M3 Solder Nut, CN3 M3 Solder Nut, J1 8 pin header, J2 8 pin socket, SW13 Switch, SW14 Switch, SW15 Switch, SW16 Switch, SW17 Switch, SW18 Switch, SW19 Switch, SW20 Switch, SW21 Switch, SW22 Switch, SW23 Switch, SW24 Switch, SW25 Switch, SW26 Switch, SW27 Switch, SW28 Switch, SW29 Switch, SW30 Switch, SW31 Switch, SW32 Switch, SW33 Switch, SW34 Switch, SW35 Switch, SW36 Switch, SW37 Switch, SW38 Switch, SW39 Switch, SW40 Switch, SW41 Switch, SW42 Switch, SW43 Switch, SW44 Switch, U2 74HC165, U3 74HC165, U4 74HC165, U5 74HC165

Commit message: Rev 1 PCBs ordered
Parts:
- added R45: 10k, Resistor_SMD:R_0402_1005Metric, F.Cu at (34.8, 71.9)
- H11, H12: value MountingHole -> M5 Mounting Hole
- P1: value ~ -> IDC Connector
Connections:
- J1 pad 2: +5V -> /RAIL_SENSE
- J2 pad 2: +5V -> /RAIL_SENSE
- P1 pad 2: +5V -> /RAIL_SENSE
Routing:
- net /RAIL_SENSE: track 0.00 -> 254.9 mm, vias 0 -> 1
- net /SLATCH: track 265.8 -> 261.9 mm
- net /SCLK: track 264.0 -> 260.4 mm
- net /LED_IN: track 80.8 -> 82.1 mm
- net Earth: vias 52 -> 77
- net +5V: vias 65 -> 61
Other:
- board text added: "+5V"
- board text added: "SmartReel Rev 1"
- board text added: "Terminate SDI"
